File: case/fr4/silk/lk23m-plate-silk.kicad_pcb (KiCad board)
At the start: 2 copper layers, 76.2 x 119.1 mm, 8 parts

Commit message: Add clearance for OLED screen to plate
Parts:
- added OL1: OLED_I2C_SSD1306, LKBD_OLED:OLED_SSD1306_128x32_0.91inch_I2C_btmSilk, F.Cu at (66.7, 38.1)
Other:
- outline, holes or cut-outs redrawn
